Commit message: first stand

File: resources/robots/h1/urdf/h1.urdf (robot description, URDF)
Before this commit: robot h1_description, 22 links, 21 joints
Joints:
- joint left_elbow_joint: type fixed -> revolute
- joint left_shoulder_pitch_joint: type fixed -> revolute
- joint left_shoulder_roll_joint: type fixed -> revolute
- joint left_shoulder_yaw_joint: type fixed -> revolute
- joint right_elbow_joint: type fixed -> revolute
- joint right_shoulder_pitch_joint: type fixed -> revolute
- joint right_shoulder_roll_joint: type fixed -> revolute
- joint right_shoulder_yaw_joint: type fixed -> revolute
- joint torso_joint: type fixed -> revolute
